File: documentation/Hardware IPSTUBE/KiCAD - Unfinished Schematics/Test1.kicad_sch (KiCad schematic)
At the start: 67 parts, among them J1 Conn_Coaxial_Small, P1 USB_C_Plug, Q2 AO3401A, SW1 Reset Switch, U1 CH340N, U2 ESP32-PICO-D4, U4 DS1302Z+, U5 AT25SF081-SSHD-X, U6 MI6118, X1 Crystal, X3 Crystal

Commit message: Fixed schematics again
Connections:
- net at Q2.1 (G), R5.1, R6.1: no longer R5.2, U2.24 (IO4)
- new net: R5.2, U2.24 (IO4)
Other:
- moved on the sheet: R5
Changed lines of the file:
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@@
 	)
 	(junction
-		(at 148.59 -49.53)
-		(diameter 0)
-		(color 0 0 0 0)
-	)
-	(junction
 		(at 38.1 -21.59)
 		(diameter 0)
@@
 	)
 	(junction
-		(at 231.14 153.67)
+		(at 140.97 -49.53)
 		(diameter 0)
 		(color 0 0 0 0)
 	)
 	(junction
-		(at 107.95 102.87)
+		(at 231.14 153.67)
 		(diameter 0)
 		(color 0 0 0 0)
 	)
 	(junction
-		(at 140.97 -49.53)
+		(at 107.95 102.87)
 		(diameter 0)
 		(color 0 0 0 0)
@@
 	)
 	(junction
-		(at 148.59 -53.34)
-		(diameter 0)
-		(color 0 0 0 0)
-	)
-	(junction
 		(at 50.8 17.78)
 		(diameter 0)
@@
 	(wire
 		(pts
+			(xy 148.59 -49.53) (xy 140.97 -49.53)
+		)
+		(stroke
+			(width 0)
+			(type default)
+		)
+	)
+	(wire
+		(pts
 			(xy 255.27 105.41) (xy 248.92 105.41)
 		)
@@
 	(wire
 		(pts
-			(xy 148.59 -49.53) (xy 148.59 29.21)
-		)
-		(stroke
-			(width 0)
-			(type default)
-		)
-	)
-	(wire
-		(pts
 			(xy 222.25 26.67) (xy 222.25 30.48)
 		)
@@
 	(wire
 		(pts
-			(xy 148.59 -60.96) (xy 148.59 -53.34)
-		)
-		(stroke
-			(width 0)
-			(type default)
-		)
-	)
-	(wire
-		(pts
 			(xy 275.59 30.48) (xy 275.59 35.56)
 		)
@@
 	(wire
 		(pts
+			(xy 148.59 -33.02) (xy 148.59 29.21)
+		)
+		(stroke
+			(width 0)
+			(type default)
+		)
+	)
+	(wire
+		(pts
 			(xy 38.1 -21.59) (xy 38.1 -41.91)
 		)
@@
 	(wire
 		(pts
+			(xy 148.59 -40.64) (xy 148.59 -49.53)
+		)
+		(stroke
+			(width 0)
+			(type default)
+		)
+	)
+	(wire
+		(pts
 			(xy 278.13 111.76) (xy 278.13 24.13)
 		)
@@
 	(wire
 		(pts
-			(xy 140.97 -49.53) (xy 148.59 -49.53)
-		)
-		(stroke
-			(width 0)
-			(type default)
-		)
-	)
-	(wire
-		(pts
 			(xy 213.36 149.86) (xy 213.36 158.75)
 		)
@@
 	(wire
 		(pts
-			(xy 148.59 -53.34) (xy 148.59 -49.53)
-		)
-		(stroke
-			(width 0)
-			(type default)
-		)
-	)
-	(wire
-		(pts
 			(xy 234.95 30.48) (xy 234.95 22.86)
 		)
@@
 	(symbol
 		(lib_id "Device:R")
-		(at 148.59 -57.15 0)
+		(at 148.59 -36.83 0)
 		(unit 1)
 		(exclude_from_sim no)
@@
 		(fields_autoplaced yes)
 		(property "Reference" "R5"
-			(at 151.13 -58.4201 0)
+			(at 151.13 -38.1001 0)
 			(effects
 				(font
@@
 		)
 		(property "Value" "1K"
-			(at 151.13 -55.8801 0)
+			(at 151.13 -35.5601 0)
 			(effects
 				(font
@@
 		)
 		(property "Footprint" ""
-			(at 146.812 -57.15 90)
+			(at 146.812 -36.83 90)
 			(effects
 				(font
@@
 		)
 		(property "Datasheet" "~"
-			(at 148.59 -57.15 0)
+			(at 148.59 -36.83 0)
 			(effects
 				(font
@@
 		)
 		(property "Description" "Resistor"
-			(at 148.59 -57.15 0)
+			(at 148.59 -36.83 0)
 			(effects
 				(font
